File: hardware/ble-key.kicad_sch (KiCad schematic)
At the start: 37 parts, among them J1 USB4105-GF-A, J2 SJ-3523-SMT, J3 JST PH battery, J4 SWD, SW1 reset, U1 MDBT50Q-1MV2, U2 BQ24074RGTR, U3 USBLC6-2SC6, Y1 32.768k

Commit message: feat: first routed layout of the nRF52840 board
46 x 26 mm, 2 layers, AISLER 2-layer ENIG rules. gen_board.py places the
footprints from the schematic's netlist and adds the outline, mounting
holes, ground pours and an antenna keep-out; route.py autoroutes with
Freerouting in Docker and refills the pours. DRC: no errors, no unconnected
pads. Dah and the charge signal moved to outer module pads, passives to 0402.

Co-Authored-By: Claude Opus 5.5 <noreply@anthropic.com>
Parts:
- C1, C10, C4, C7, C9: footprint Capacitor_SMD:C_0603_1608Metric -> Capacitor_SMD:C_0402_1005Metric
- R1, R10, R11, R12, R13, R14, R15, R2, R3, R4, R5, R6, R7, R8, R9: footprint Resistor_SMD:R_0603_1608Metric -> Resistor_SMD:R_0402_1005Metric
Connections:
- net DAH: now also U1.22 (P0.06); no longer U1.21 (P0.05)
- net ~{CHG}: now also U1.12 (P0.31); no longer U1.13 (P0.28)

Commit message: feat: part numbers for the crystal, its capacitors and the DC/DC inductor
Y1 Epson FC-12M (CL 9 pF, matched to the 12 pF capacitors per Nordic's
guidance), C9/C10 Murata GRM1555C1H120GA01D, L1 Taiyo Yuden LBMF1608T100K as
on the nRF52840-DK. The board's footprints now carry the MPN field too, so
AISLER can match parts from the layout file.

Co-Authored-By: Claude Opus 5.5 <noreply@anthropic.com>
Parts:
- C10, C9: MPN (none) -> GRM1555C1H120GA01D
- L1: MPN (none) -> LBMF1608T100K
- Y1: MPN (none) -> FC-12M 32.7680KA-AC0
Changed lines of the file:
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@@
   (property "Footprint" "Inductor_SMD:L_0603_1608Metric" (at 238.76 175.26 0) (effects (font (size 1.27 1.27)) (hide yes)))
   (property "Datasheet" "" (at 238.76 175.26 0) (effects (font (size 1.27 1.27)) (hide yes)))
+  (property "MPN" "LBMF1608T100K" (at 238.76 175.26 0) (effects (font (size 1.27 1.27)) (hide yes)))
   (pin "1")
   (pin "2")
@@
   (property "Footprint" "Crystal:Crystal_SMD_2012-2Pin_2.0x1.2mm" (at 254.0 160.02 0) (effects (font (size 1.27 1.27)) (hide yes)))
   (property "Datasheet" "" (at 254.0 160.02 0) (effects (font (size 1.27 1.27)) (hide yes)))
+  (property "MPN" "FC-12M 32.7680KA-AC0" (at 254.0 160.02 0) (effects (font (size 1.27 1.27)) (hide yes)))
   (pin "1")
   (pin "2")
@@
   (property "Footprint" "Capacitor_SMD:C_0402_1005Metric" (at 248.92 175.26 0) (effects (font (size 1.27 1.27)) (hide yes)))
   (property "Datasheet" "" (at 248.92 175.26 0) (effects (font (size 1.27 1.27)) (hide yes)))
+  (property "MPN" "GRM1555C1H120GA01D" (at 248.92 175.26 0) (effects (font (size 1.27 1.27)) (hide yes)))
   (pin "1")
   (pin "2")
@@
   (property "Footprint" "Capacitor_SMD:C_0402_1005Metric" (at 259.08 175.26 0) (effects (font (size 1.27 1.27)) (hide yes)))
   (property "Datasheet" "" (at 259.08 175.26 0) (effects (font (size 1.27 1.27)) (hide yes)))
+  (property "MPN" "GRM1555C1H120GA01D" (at 259.08 175.26 0) (effects (font (size 1.27 1.27)) (hide yes)))
   (pin "1")
   (pin "2")

Commit message: feat: JLCPCB production files with LCSC part numbers
export_jlc.py writes zipped Gerbers and drill files, a BOM in JLCPCB's format
and a placement file from the board, with the LCSC part numbers now stored in
the schematic. The module and the reset switch are out of stock at JLCPCB.

Co-Authored-By: Claude Opus 5.5 <noreply@anthropic.com>
Parts:
- C1: LCSC (none) -> C52923
- C10, C9: LCSC (none) -> C1547
- C2, C3: LCSC (none) -> C19666
- C4, C7: LCSC (none) -> C1525
- C5, C6, C8: LCSC (none) -> C19702
- D1: LCSC (none) -> C2286
- D2: LCSC (none) -> C2986058
- J1: LCSC (none) -> C5184243
- J2: LCSC (none) -> C4991872
- J3: LCSC (none) -> C295747
- L1: LCSC (none) -> C87216
- R1, R2, R5: LCSC (none) -> C25905
- R10, R11: LCSC (none) -> C25117
- R12, R13: LCSC (none) -> C11702
- R14, R15: LCSC (none) -> C25100
- R3: LCSC (none) -> C25744
- R4: LCSC (none) -> C11460
- R6, R7: LCSC (none) -> C25741
- R8, R9: LCSC (none) -> C26083
- SW1: LCSC (none) -> C79174
- U1: LCSC (none) -> C5118826
- U2: LCSC (none) -> C54313
- U3: LCSC (none) -> C7519
- Y1: LCSC (none) -> C96341
